Commit message: prueba motor CCW , ya vuela bien

File: models/7in_3blades_v2/HELICE_PRUEBA.urdf (robot description, URDF)
Before this commit: robot HELICE_PRUEBA, 1 links, 0 joints
Links:
- link Helice: geometry collision mesh filename=meshes/7in_3blades.stl scale=0.001 0.001 0.001; visual mesh filename=meshes/7in_3blades.stl scale=0.001 0.001 0.001
